Commit message: docs(sim): 模型来源署名改为 WWNT Robotics 核心模型，清除 LuwuDynamics/XgoDuck 标识

File: sim/wwduck/urdf/XGODUCK.urdf (robot description, URDF)
Before this commit: robot xgoduck_v2, 15 links, 14 joints
Links:
- link head_pitch: geometry collision mesh filename=package://wwduck/meshes/head_pitch.STL; visual mesh filename=package://wwduck/meshes/head_pitch.STL
- link head_roll: geometry collision mesh filename=package://wwduck/meshes/head_roll.STL; visual mesh filename=package://wwduck/meshes/head_roll.STL
- link head_yaw: geometry collision mesh filename=package://wwduck/meshes/head_yaw.STL; visual mesh filename=package://wwduck/meshes/head_yaw.STL
- link left_ankle: geometry collision mesh filename=package://wwduck/meshes/left_ankle.STL; visual mesh filename=package://wwduck/meshes/left_ankle.STL
- link left_hip_pitch: geometry collision mesh filename=package://wwduck/meshes/left_hip_pitch.STL; visual mesh filename=package://wwduck/meshes/left_hip_pitch.STL
- link left_hip_roll: geometry collision mesh filename=package://wwduck/meshes/left_hip_roll.STL; visual mesh filename=package://wwduck/meshes/left_hip_roll.STL
- link left_hip_yaw: geometry collision mesh filename=package://wwduck/meshes/left_hip_yaw.STL; visual mesh filename=package://wwduck/meshes/left_hip_yaw.STL
- link left_knee: geometry collision mesh filename=package://wwduck/meshes/left_knee.STL; visual mesh filename=package://wwduck/meshes/left_knee.STL
- link neck_pitch: geometry collision mesh filename=package://wwduck/meshes/neck_pitch.STL; visual mesh filename=package://wwduck/meshes/neck_pitch.STL
- link right_ankle: geometry collision mesh filename=package://wwduck/meshes/right_ankle.STL; visual mesh filename=package://wwduck/meshes/right_ankle.STL
- link right_hip_pitch: geometry collision mesh filename=package://wwduck/meshes/right_hip_pitch.STL; visual mesh filename=package://wwduck/meshes/right_hip_pitch.STL
- link right_hip_roll: geometry collision mesh filename=package://wwduck/meshes/right_hip_roll.STL; visual mesh filename=package://wwduck/meshes/right_hip_roll.STL
- link right_hip_yaw: geometry collision mesh filename=package://wwduck/meshes/right_hip_yaw.STL; visual mesh filename=package://wwduck/meshes/right_hip_yaw.STL
- link right_knee: geometry collision mesh filename=package://wwduck/meshes/right_knee.STL; visual mesh filename=package://wwduck/meshes/right_knee.STL
- link trunk_base: geometry collision mesh filename=package://wwduck/meshes/trunk_base.STL; visual mesh filename=package://wwduck/meshes/trunk_base.STL
